Commit message: Corrected the URDF to adjust joints

File: install/Industrial_description/share/Industrial_description/urdf/Industrial.xacro (robot description, xacro)
@@ -91,5 +91,5 @@
   </inertial>
   <visual>
-    <origin xyz="0.194373 0.460509 -0.650413" rpy="0 0 0"/>
+    <origin xyz="0.208 0.460509 -0.650413" rpy="0 0 0"/>
     <geometry>
       <mesh filename="file://$(find Industrial_description)/meshes/Jaw_4_1.stl" scale="0.001 0.001 0.001"/>
@@ -131,5 +131,5 @@
   </inertial>
   <visual>
-    <origin xyz="0.187341 0.677117 -0.650413" rpy="0 0 0"/>
+    <origin xyz="0.209 0.677117 -0.65" rpy="0 0 0"/>
     <geometry>
       <mesh filename="file://$(find Industrial_description)/meshes/Jaw_6_1.stl" scale="0.001 0.001 0.001"/>
@@ -151,5 +151,5 @@
   </inertial>
   <visual>
-    <origin xyz="0.226983 0.711408 -0.663413" rpy="0 0 0"/>
+    <origin xyz="0.25 0.711408 -0.663413" rpy="0 0 0"/>
     <geometry>
       <mesh filename="file://$(find Industrial_description)/meshes/Jaw_7_copy_1.stl" scale="0.001 0.001 0.001"/>
@@ -171,5 +171,5 @@
   </inertial>
   <visual>
-    <origin xyz="0.145413 0.708571 -0.663413" rpy="0 0 0"/>
+    <origin xyz="0.17 0.708571 -0.663413" rpy="0 0 0"/>
     <geometry>
       <mesh filename="file://$(find Industrial_description)/meshes/Jaw_7_copy_2.stl" scale="0.001 0.001 0.001"/>
@@ -205,5 +205,5 @@
 </joint>
 <joint name="L3_L4" type="continuous">
-  <origin xyz="0.056521 -0.244183 0.045" rpy="0 0 0"/>
+  <origin xyz="0.0425 -0.244183 0.0425" rpy="0 0 0"/>
   <parent link="Jaw_3_1"/>
   <child link="Jaw_4_1"/>
@@ -211,5 +211,5 @@
 </joint>
 <joint name="L4_L5" type="revolute">
-  <origin xyz="-0.008228 -0.123082 0.0" rpy="0 0 0"/>
+  <origin xyz="0.005 -0.123082 0.0" rpy="0 0 0"/>
   <parent link="Jaw_4_1"/>
   <child link="Jaw_5_1"/>
@@ -218,9 +218,10 @@
 </joint>
 <joint name="L5_L6" type="continuous">
-  <origin xyz="0.01526 -0.093526 0.0" rpy="0 0 0"/>
+  <origin xyz="-0.005 -0.093526 0.0" rpy="0 0 0"/>
   <parent link="Jaw_5_1"/>
   <child link="Jaw_6_1"/>
-  <axis xyz="-0.034755 0.999396 0.0"/>
-</joint>
+  <axis xyz="0.0 1.0 0.0"/>
+</joint>
+<!--  -->
 <joint name="L6_GL" type="revolute">
   <origin xyz="-0.039642 -0.034291 0.013" rpy="0 0 0"/>
@@ -235,5 +236,5 @@
   <child link="Jaw_7_copy_2"/>
   <axis xyz="-0.0 -0.0 -1.0"/>
-  <limit upper="5.235988" lower="4.712389" effort="100" velocity="100"/>
+  <limit upper="-1.0" lower="0.042" effort="100" velocity="100"/>
 </joint>
 </robot>
